File: eval/SKY130_PLL_eval_PCB/SKY130_PLL_eval.kicad_pcb (KiCad board)
At the start: 4 copper layers, 56.2 x 87.2 mm, 44 parts, among them J1 Conn_02x10_Odd_Even, J2 Conn_02x03_Odd_Even, J3 Conn_02x07_Odd_Even, J5 Conn_02x07_Odd_Even, J6 Conn_02x06_Odd_Even, U1 ADM7154ARDZ-1.8-R7, U2 Caravel_QFN

Commit message: minor layout changes
Parts:
- moved J_PLL_REF_IN1 0.77 mm to (134.0, 71.3)
Routing:
- net flash_io1_arty: track 28.3 -> 31.2 mm
- net /PLL_IO/pll_sma_in: track 8.92 -> 11.6 mm
- net flash_io2_arty: track 29.3 -> 31.9 mm
- net flash_clk_arty: track 28.4 -> 30.2 mm
- net flash_csb_arty: track 27.5 -> 28.5 mm
- net GND: vias 534 -> 536
